File: snappergps_board_2_1_0.sch (EAGLE design)
At the start: 66 parts, among them IC1 W25N512GVEIG_W25N512GVEIG, J1 DX07S016JA1R1500, J4 2996TR_2996TR2996TR-CREAM, J5 2996TR_2996TR2996TR-CREAM, Q1 TT8M1TRAMANDA, Q3 TT8M1TRAMANDA, Q4 TT8M1TRAMANDA, U1 EFM32HG310F64, U2 RF_CIRCUIT-SE4150L, U3 TVS_DIODE-PRTR5V0U2AX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

Commit message: Tweak schematic
Other:
- note removed: "Using Al's desgin as inspiration: https://github.com/arribada/horizon/blob/master/hardware/horizon_v4_1/"
Changed lines of the file:
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@@
 <part name="FRAME1" library="SparkFun-Aesthetics" deviceset="FRAME-A4L" device="">
 <attribute name="CNAME" value="RF front end"/>
-<attribute name="CREVISION" value="2.9"/>
+<attribute name="CREVISION" value="2.1.0"/>
 <attribute name="DESIGNER" value="A. Rogers, J. Beuchert"/>
 <attribute name="REV" value="2.4"/>
@@
 <part name="FRAME2" library="SparkFun-Aesthetics" deviceset="FRAME-A4L" device="">
 <attribute name="CNAME" value="Flash, power, LEDs, and LFXTAL"/>
-<attribute name="CREVISION" value="2.9"/>
+<attribute name="CREVISION" value="2.1.0"/>
 <attribute name="DESIGNER" value="A. Rogers, J. Beuchert"/>
 </part>
 <part name="FRAME3" library="SparkFun-Aesthetics" deviceset="FRAME-A4L" device="">
 <attribute name="CNAME" value="USB and power"/>
-<attribute name="CREVISION" value="2.9"/>
+<attribute name="CREVISION" value="2.1.0"/>
 <attribute name="DESIGNER" value="A. Rogers, J. Beuchert"/>
 </part>
 <part name="FRAME4" library="SparkFun-Aesthetics" deviceset="FRAME-A4L" device="">
 <attribute name="CNAME" value="MCU IO connections"/>
-<attribute name="CREVISION" value="2.9"/>
+<attribute name="CREVISION" value="2.1.0"/>
 <attribute name="DESIGNER" value="A. Rogers"/>
 </part>
@@
 <sheet>
 <plain>
-<text x="-251.46" y="231.14" size="1.778" layer="91">Using Al's desgin as inspiration:
-https://github.com/arribada/horizon/blob/master/hardware/horizon_v4_1/</text>
 <text x="-251.46" y="226.06" size="1.778" layer="91">SnapperGPS zebra logo</text>
 </plain>
@@
 </drawing>
 <compatibility>
-<note version="6.3" minversion="6.2.2" severity="warning">
-Since Version 6.2.2 text objects can contain more than one line,
-which will not be processed correctly with this version.
-</note>
 <note version="8.2" severity="warning">
 Since Version 8.2, EAGLE supports online libraries. The ids
